Commit message: Adding debug blocks to prop the sim model up while testing controls

File: ros_workspace/src/robomagellan_2024_description/urdf/robomagellan_2024.urdf.xacro (robot description, xacro)
@@ -144,4 +144,29 @@
       <origin rpy="0 0 0" xyz="0.38735 0 0.0381"/>
     </visual>
+    <!-- Debug Blocks -->
+    <visual name="front_debug_block_visual">
+      <geometry>
+        <box size="0.0508 0.0508 0.0508"/>
+      </geometry>
+      <origin rpy="0 0 0" xyz="0.38735 0 -0.0635"/>
+    </visual>
+    <collision name="front_debug_block_collision">
+      <geometry>
+        <box size="0.0508 0.0508 0.0508"/>
+      </geometry>
+      <origin rpy="0 0 0" xyz="0.38735 0 -0.0635"/>
+    </collision>
+    <visual name="rear_debug_block_visual">
+      <geometry>
+        <box size="0.0508 0.0508 0.0508"/>
+      </geometry>
+      <origin rpy="0 0 0" xyz="-0.38735 0 -0.0635"/>
+    </visual>
+    <collision name="rear_debug_block_collision">
+      <geometry>
+        <box size="0.0508 0.0508 0.0508"/>
+      </geometry>
+      <origin rpy="0 0 0" xyz="-0.38735 0 -0.0635"/>
+    </collision>
   </link>
   <!-- Wheels -->
