Commit message: Updating Robomagellan URDF and ROS 2 Gazebo Sim Launch
This commit corrects the Robomagellan URDF to have the proper TF frames
such as `base_footprint` and `base_link`.  The inertial matrix for the
wheels was also fixed.  Finally, a Python launch file is added to launch
the Gazebo sim, process the URDF file, and spawn the simulated robot.

Signed-off-by: Bryant Pong <rcxking@gmail.com>

File: ros2_ws/src/robomagellan_description/description/robomagellan.urdf.xacro (robot description, xacro)
@@ -1,158 +1,5 @@
-<?xml version="1.0" ?>
-<robot name="robomagellan_2024" xmlns:xacro="http://ros.org/wiki/xacro">
-  <!--
-    Robot mechanical dimensions.
-    Main chassis frame consists of 2 side bars and 2 front/rear bars with the
-    following dimensions:
-    Side Bars:
-    Length: 29.5 inches/0.7493 meters
-    Width: 1 inch/0.0254 meters
-    Height: 2 inches/0.0508 meters
-    Front/Rear Bars:
-    Length: 25 inches/0.635 meters
-    Width: 1 inch/0.0254 meters
-    Height: 2 inches/0.0508 meters
-    Wheels:
-    Diameter: 6 inches/0.1524 meters
-    Width: 1.775 inches/0.045085 meters
-  -->
-  <xacro:property name="sidebar_length" value="0.7493"/>
-  <xacro:property name="sidebar_width" value="0.0254"/>
-  <xacro:property name="sidebar_height" value="0.0508"/>
-  <xacro:property name="sidebar_y_offset" value="0.20955"/>
-  <xacro:property name="frontbar_length" value="0.635"/>
-  <xacro:property name="frontbar_width" value="0.0254"/>
-  <xacro:property name="frontbar_height" value="0.0508"/>
-  <xacro:property name="frontbar_x_offset" value="0.38735"/>
-  <xacro:property name="wheel_radius" value="0.0762"/>
-  <xacro:property name="wheel_width" value="0.045085"/>
-  <xacro:property name="wheel_mass" value="0.36196671"/>
-  <xacro:property name="wheel_x_offset" value="0.28575"/>
-  <xacro:property name="wheel_y_offset" value="0.2447925"/>
-  <!-- Macro to create the side bars -->
-  <xacro:macro name="sidebar" params="prefix reflect">
-    <visual name="${prefix}_side_visual">
-      <origin xyz="0 ${sidebar_y_offset*reflect} 0" rpy="0 0 0"/>
-      <geometry>
-        <box size="${sidebar_length} ${sidebar_width} ${sidebar_height}"/>
-      </geometry>
-    </visual>
-    <collision name="${prefix}_side_collision">
-      <origin xyz="0 ${sidebar_y_offset*reflect} 0" rpy="0 0 0"/>
-      <geometry>
-        <box size="${sidebar_length} ${sidebar_width} ${sidebar_height}"/>
-      </geometry>
-    </collision>
-  </xacro:macro>
-  <!-- Macro to create the front/rear bars -->
-  <xacro:macro name="frontbar" params="prefix reflect">
-    <visual name="${prefix}_visual">
-      <origin xyz="${frontbar_x_offset*reflect} 0 0" rpy="0 0 1.5708"/>
-      <geometry>
-        <box size="${frontbar_length} ${frontbar_width} ${frontbar_height}"/>
-      </geometry>
-    </visual>
-    <collision name="${prefix}_collision">
-      <origin xyz="${frontbar_x_offset*reflect} 0 0" rpy="0 0 1.5708"/>
-      <geometry>
-        <box size="${frontbar_length} ${frontbar_width} ${frontbar_height}"/>
-      </geometry>
-    </collision>
-  </xacro:macro>
-  <!-- Macro to create the wheels -->
-  <xacro:macro name="wheel" params="prefix suffix reflectx reflecty">
-    <link name="${prefix}_${suffix}_wheel">
-      <inertial>
-        <mass value="${wheel_mass}"/>
-        <inertia ixx="0.0005867" iyy="0.0005867" izz="0.0010509" ixy="0.0" ixz="0.0" iyz="0.0"/>
-      </inertial>
-      <visual>
-        <geometry>
-          <cylinder length="${wheel_width}" radius="${wheel_radius}"/>
-        </geometry>
-       <material name="black"/>
-        <origin rpy="1.5708 0 0" xyz="0 0 0"/>
-      </visual>
-      <collision>
-        <geometry>
-          <cylinder length="${wheel_width}" radius="${wheel_radius}"/>
-        </geometry>
-        <origin rpy="1.5708 0 0" xyz="0 0 0"/>
-      </collision>
-    </link>
-    <!-- Joint connecting this wheel to the base_link -->
-    <joint name="${prefix}_${suffix}_joint" type="continuous">
-      <axis xyz="0 1 0" rpy="0 0 0"/>
-      <parent link="base_link"/>
-      <child link="${prefix}_${suffix}_wheel"/>
-      <origin xyz="${reflectx*wheel_x_offset} ${reflecty*wheel_y_offset} 0.0"
-              rpy="0 0 0"/>
-    </joint>
-    <!--
-      This block provides Gazebo with information on the wheel's physical
-      properties.
-    -->
-    <gazebo reference="${prefix}_${suffix}_wheel">
-      <kp value="10000000.0"/>
-      <kd value="1.0"/>
-      <material>Gazebo/Black</material>
-      <!-- Friction coefficients -->
-      <mu1 value="0.001"/>
-      <mu2 value="0.001"/>
-    </gazebo>
-    <!--
-      This block connects the wheel joint to an actuator (motor), which informs
-      both the simulation and visualization of the robot.
-    -->
-    <transmission name="${prefix}_${suffix}_wheel_trans">
-      <type>transmission_interface/SimpleTransmission</type>
-      <actuator name="${prefix}_${suffix}_wheel_motor">
-        <mechanicalReduction>1</mechanicalReduction>
-      </actuator>
-      <joint name="${prefix}_${suffix}_joint">
-        <hardwareInterface>hardware_interface/VelocityJointInterface</hardwareInterface>
-      </joint>
-    </transmission>
-  </xacro:macro>
-  <material name="black">
-    <color rgba="0 0 0 1"/>
-  </material>
-  <link name="base_link">
-    <!--
-      The chassis will be represented with a cuboid with the above dimensions
-      and a weight of 50 lbs (the max limit allowed).
-    -->
-    <inertial>
-      <mass value="22.68"/>
-      <inertia ixx="0.767" iyy="1.2145" izz="1.9717" ixy="0.0" ixz="0.0" iyz="0.0"/>
-    </inertial>
-    <!-- Left/Right sidebars -->
-    <xacro:sidebar prefix="left" reflect="1"/>
-    <xacro:sidebar prefix="right" reflect="-1"/>
-    <!-- Front/Rear bars -->
-    <xacro:frontbar prefix="front" reflect="1"/>
-    <xacro:frontbar prefix="rear" reflect="-1"/>
-    <!--
-      For visualization purposes a small cube will be added to the front of the
-      robot.  No collision is used because the real robot does not have this
-      cube.
-    -->
-    <visual name="cube_visual">
-      <geometry>
-        <box size="0.0254 0.0254 0.0254"/>
-      </geometry>
-      <origin rpy="0 0 0" xyz="0.38735 0 0.0381"/>
-    </visual>
-  </link>
-  <!-- Wheels -->
-  <xacro:wheel prefix="left" suffix="front" reflectx="1" reflecty="1"/>
-  <xacro:wheel prefix="left" suffix="rear" reflectx="-1" reflecty="1"/>
-  <xacro:wheel prefix="right" suffix="front" reflectx="1" reflecty="-1"/>
-  <xacro:wheel prefix="right" suffix="rear" reflectx="-1" reflecty="-1"/>
-  <!-- Gazebo Plugin for Differential Drive Controller -->
-  <gazebo>
-    <plugin name="gazebo_ros_control" filename="libgazebo_ros_control.so">
-      <robotNamespace>/</robotNamespace>
-    </plugin>
-  </gazebo>
+<?xml version="1.0"?>
+<robot xmlns:xacro="http://www.ros.org/wiki/xacro" name="robot">
+  <xacro:arg name="sim_mode" default="false"/>
+  <xacro:include filename="robomagellan_core.urdf.xacro"/>
 </robot>
