Commit message: robomagellan_description Upgrades
This commit upgrades `robomagellan_description` to update the URDF files
and creates RVIZ/new launch files that work with ROS 2 Jazzy.

Signed-off-by: Bryant Pong <rcxking@gmail.com>

File: ros2_ws/src/robomagellan_description/urdf/robomagellan.urdf.xacro (robot description, xacro)
@@ -1,4 +1,10 @@
 <?xml version="1.0"?>
-<robot xmlns:xacro="http://www.ros.org/wiki/xacro">
+<robot name="robot" xmlns:xacro="http://www.ros.org/wiki/xacro">
+  <!-- Load simulated or real hardware interfaces -->
+  <xacro:arg name="is_sim" default="true"/>
+  <!-- Include Gazebo parameters -->
+ <!-- <xacro:include filename="$(find robomagellan_description)/urdf/gazebo.xacro"/> -->
+  <!-- Include ros2_contol plugins -->
+ <!-- <xacro:include filename="$(find robomagellan_description)/urdf/ros2_control.xacro"/> -->
   <!-- Inertial Macros -->
   <xacro:macro name="inertial_box" params="mass x y z">
@@ -83,4 +89,5 @@
       <xacro:inertial_cylinder mass="${wheel_mass}" length="${wheel_width}" radius="${wheel_radius}"/>
       <visual>
+        <origin xyz="0 0 0" rpy="${-reflecty*pi/2} 0 0"/>
         <geometry>
           <cylinder length="${wheel_width}" radius="${wheel_radius}"/>
@@ -89,4 +96,5 @@
       </visual>
       <collision>
+        <origin xyz="0 0 0" rpy="${-reflecty*pi/2} 0 0"/>
         <geometry>
           <cylinder length="${wheel_width}" radius="${wheel_radius}"/>
@@ -96,9 +104,8 @@
     <!-- Joint connecting this wheel to the base_link -->
     <joint name="${prefix}_${suffix}_joint" type="continuous">
-      <axis xyz="0 0 1" rpy="0 0 0"/>
+      <origin xyz="${reflectx*wheel_x_offset} ${reflecty*wheel_y_offset} 0" rpy="0 0 0"/>
       <parent link="base_link"/>
       <child link="${prefix}_${suffix}_wheel"/>
-      <origin xyz="${reflectx*wheel_x_offset} ${reflecty*wheel_y_offset} 0.0"
-              rpy="${-reflecty*pi/2} 0 0"/>
+      <axis xyz="0 1 0"/>
     </joint>
   </xacro:macro>
@@ -107,4 +114,5 @@
       <xacro:inertial_cylinder mass="${wheel_mass}" length="${wheel_width}" radius="${wheel_radius}"/>
       <visual>
+        <origin xyz="0 0 0" rpy="${-reflecty*pi/2} 0 0"/>
         <geometry>
           <cylinder length="${wheel_width}" radius="${wheel_radius}"/>
@@ -113,4 +121,5 @@
       </visual>
       <collision>
+        <origin xyz="0 0 0" rpy="${-reflecty*pi/2} 0 0"/>
         <geometry>
           <cylinder length="${wheel_width}" radius="${wheel_radius}"/>
@@ -120,9 +129,8 @@
     <!-- Joint connecting this wheel to the base_link -->
     <joint name="${prefix}_${suffix}_joint" type="continuous">
-      <axis xyz="0 0 1" rpy="0 0 0"/>
+      <origin xyz="${reflectx*wheel_x_offset} ${reflecty*wheel_y_offset} 0" rpy="0 0 0"/>
       <parent link="base_link"/>
       <child link="${prefix}_${suffix}_wheel"/>
-      <origin xyz="${reflectx*wheel_x_offset} ${reflecty*wheel_y_offset} 0.0"
-              rpy="${-reflecty*pi/2} 0 0"/>
+      <axis xyz="0 1 0"/>
       <mimic joint="${prefix}_front_joint" multiplier="1.0" offset="0.0"/>
     </joint>
@@ -131,16 +139,8 @@
     <color rgba="0 0 0 1"/>
   </material>
-  <!-- Base Link -->
-  <link name="base_link"/>
-  <!-- Base Footprint Link -->
+  <!-- Base Footprint Link.  This is the 2D ground projection of base_link -->
   <link name="base_footprint"/>
-  <!-- Attach Base Link to Base Footprint -->
-  <joint name="base_footprint_joint" type="fixed">
-    <parent link="base_link"/>
-    <child link="base_footprint"/>
-    <origin xyz="0 0 0" rpy="0 0 0"/>
-  </joint>
-  <!-- Chassis represented by a 50 lbs cuboid (max weight limit) -->
-  <link name="chassis">
+  <!-- Base link represented by a 50 lbs cuboid (max weight limit) -->
+  <link name="base_link">
     <!-- Left/Right sidebars -->
     <xacro:sidebar prefix="left" reflect="1"/>
@@ -162,8 +162,10 @@
     <xacro:inertial_box mass="${robot_mass}" x="${sidebar_length+2*frontbar_width}" y="${frontbar_length}" z="${sidebar_height}"/>
   </link>
-  <!-- Attach chassis to Base Link -->
-  <joint name="chassis_joint" type="fixed">
-    <parent link="base_link"/>
-    <child link="chassis"/>
+  <!-- Attach base_link to base_footprint -->
+  <joint name="base_joint" type="fixed">
+    <parent link="base_footprint"/>
+    <child link="base_link"/>
+    <!-- base_link is center of the chassis, so need to shift +Z by wheel radius -->
+    <origin xyz="0 0 ${wheel_radius}" rpy="0 0 0"/>
   </joint>
   <!-- Wheels -->

Commit message: robomagellan_description - Updating URDF Wheels
This commit updates the `robomagellan.urdf.xacro` to correct the wheels'
inertial matrices and change the wheels' collision layers to spheres
from cylinders.

Signed-off-by: Bryant Pong <rcxking@gmail.com>

File: ros2_ws/src/robomagellan_description/urdf/robomagellan.urdf.xacro (robot description, xacro)
@@ -16,10 +16,11 @@
     </inertial>
   </xacro:macro>
-  <xacro:macro name="inertial_cylinder" params="mass length radius">
+  <!-- Wheels are rotated 90 degrees about x-axis -->
+  <xacro:macro name="inertial_cylinder" params="mass radius height">
     <inertial>
       <mass value="${mass}"/>
-      <inertia ixx="${(1/12) * mass * (3*radius*radius + length*length)}" ixy="0.0" ixz="0.0"
-               iyy="${(1/12) * mass * (3*radius*radius + length*length)}" iyz="0.0"
-               izz="${(1/2) * mass * (radius*radius)}"/>
+      <inertia ixx="${(1/12) * mass * (3*radius*radius + height*height)}" ixy="0.0" ixz="0.0"
+               iyy="${(1/2) * mass * (radius*radius)}" iyz="0.0"
+               izz="${(1/12) * mass * (3*radius*radius + height*height)}"/>
     </inertial>
   </xacro:macro>
@@ -87,5 +88,5 @@
   <xacro:macro name="wheel" params="prefix suffix reflectx reflecty">
     <link name="${prefix}_${suffix}_wheel">
-      <xacro:inertial_cylinder mass="${wheel_mass}" length="${wheel_width}" radius="${wheel_radius}"/>
+      <xacro:inertial_cylinder mass="${wheel_mass}" height="${wheel_width}" radius="${wheel_radius}"/>
       <visual>
         <origin xyz="0 0 0" rpy="${-reflecty*pi/2} 0 0"/>
@@ -97,6 +98,7 @@
       <collision>
         <origin xyz="0 0 0" rpy="${-reflecty*pi/2} 0 0"/>
+        <!-- Use a sphere for collisions to have one ground contact point -->
         <geometry>
-          <cylinder length="${wheel_width}" radius="${wheel_radius}"/>
+          <sphere radius="${wheel_radius}"/>
         </geometry>
       </collision>
@@ -112,5 +114,5 @@
   <xacro:macro name="mimic_wheel" params="prefix suffix reflectx reflecty">
     <link name="${prefix}_${suffix}_wheel">
-      <xacro:inertial_cylinder mass="${wheel_mass}" length="${wheel_width}" radius="${wheel_radius}"/>
+      <xacro:inertial_cylinder mass="${wheel_mass}" height="${wheel_width}" radius="${wheel_radius}"/>
       <visual>
         <origin xyz="0 0 0" rpy="${-reflecty*pi/2} 0 0"/>
@@ -122,6 +124,7 @@
       <collision>
         <origin xyz="0 0 0" rpy="${-reflecty*pi/2} 0 0"/>
+        <!-- Use a sphere for collisions to have one ground contact point -->
         <geometry>
-          <cylinder length="${wheel_width}" radius="${wheel_radius}"/>
+          <sphere radius="${wheel_radius}"/>
         </geometry>
       </collision>

Commit message: robomagellan_description - Removed mimic_wheel Macro
This commit removes the `mimic_wheel` macro and replaces it with an
additional `mimic_wheel` parameter to the `wheel` macro.

Signed-off-by: Bryant Pong <rcxking@gmail.com>

File: ros2_ws/src/robomagellan_description/urdf/robomagellan.urdf.xacro (robot description, xacro)
@@ -86,5 +86,5 @@
   </xacro:macro>
   <!-- Macro to create the wheels -->
-  <xacro:macro name="wheel" params="prefix suffix reflectx reflecty">
+  <xacro:macro name="wheel" params="prefix suffix reflectx reflecty mimic_wheel">
     <link name="${prefix}_${suffix}_wheel">
       <xacro:inertial_cylinder mass="${wheel_mass}" height="${wheel_width}" radius="${wheel_radius}"/>
@@ -110,31 +110,8 @@
       <child link="${prefix}_${suffix}_wheel"/>
       <axis xyz="0 1 0"/>
-    </joint>
-  </xacro:macro>
-  <xacro:macro name="mimic_wheel" params="prefix suffix reflectx reflecty">
-    <link name="${prefix}_${suffix}_wheel">
-      <xacro:inertial_cylinder mass="${wheel_mass}" height="${wheel_width}" radius="${wheel_radius}"/>
-      <visual>
-        <origin xyz="0 0 0" rpy="${-reflecty*pi/2} 0 0"/>
-        <geometry>
-          <cylinder length="${wheel_width}" radius="${wheel_radius}"/>
-        </geometry>
-       <material name="black"/>
-      </visual>
-      <collision>
-        <origin xyz="0 0 0" rpy="${-reflecty*pi/2} 0 0"/>
-        <!-- Use a sphere for collisions to have one ground contact point -->
-        <geometry>
-          <sphere radius="${wheel_radius}"/>
-        </geometry>
-      </collision>
-    </link>
-    <!-- Joint connecting this wheel to the base_link -->
-    <joint name="${prefix}_${suffix}_joint" type="continuous">
-      <origin xyz="${reflectx*wheel_x_offset} ${reflecty*wheel_y_offset} 0" rpy="0 0 0"/>
-      <parent link="base_link"/>
-      <child link="${prefix}_${suffix}_wheel"/>
-      <axis xyz="0 1 0"/>
-      <mimic joint="${prefix}_front_joint" multiplier="1.0" offset="0.0"/>
+      <!-- Is this a mimic wheel? -->
+      <xacro:if value="${mimic_wheel}">
+        <mimic joint="${prefix}_front_joint" multiplier="1.0" offset="0.0"/>
+      </xacro:if>
     </joint>
   </xacro:macro>
@@ -173,7 +150,7 @@
   </joint>
   <!-- Wheels -->
-  <xacro:wheel prefix="left" suffix="front" reflectx="1" reflecty="1"/>
-  <xacro:mimic_wheel prefix="left" suffix="rear" reflectx="-1" reflecty="1"/>
-  <xacro:wheel prefix="right" suffix="front" reflectx="1" reflecty="-1"/>
-  <xacro:mimic_wheel prefix="right" suffix="rear" reflectx="-1" reflecty="-1"/>
+  <xacro:wheel prefix="left" suffix="front" reflectx="1" reflecty="1" mimic_wheel="false"/>
+  <xacro:wheel prefix="left" suffix="rear" reflectx="-1" reflecty="1" mimic_wheel="true"/>
+  <xacro:wheel prefix="right" suffix="front" reflectx="1" reflecty="-1" mimic_wheel="false"/>
+  <xacro:wheel prefix="right" suffix="rear" reflectx="-1" reflecty="-1" mimic_wheel="true"/>
 </robot>
