Commit message: ros2_control - Initial Differential Drive Controller Integration
This commit adds in the launch & config files to load the stock
differential drive controller using the `ros2_control`
`controller_manager`.

This is tested using `robomagellan_bringup` `sim.launch.py`.

Signed-off-by: Bryant Pong <rcxking@gmail.com>

File: ros2_ws/src/robomagellan_description/urdf/gazebo.xacro (robot description, xacro)
@@ -1,20 +1,45 @@
 <?xml version="1.0"?>
-<robot xmlns:xacro="http://www.ros.org/wiki/xacro">
+<robot name="robot" xmlns:xacro="http://www.ros.org/wiki/xacro">
+  <!-- Wheel links -->
+  <gazebo reference="left_front_wheel">
+    <mu1>1000000000000000.0</mu1>
+    <mu2>1000000000000000.0</mu2>
+    <kp>1000000000000.0</kp>
+    <kd>10.0</kd>
+    <minDepth>0.001</minDepth>
+    <maxVel>0.1</maxVel>
+    <fdir1>1 0 0</fdir1>
+  </gazebo>
+  <gazebo reference="right_front_wheel">
+    <mu1>1000000000000000.0</mu1>
+    <mu2>1000000000000000.0</mu2>
+    <kp>1000000000000.0</kp>
+    <kd>10.0</kd>
+    <minDepth>0.001</minDepth>
+    <maxVel>0.1</maxVel>
+    <fdir1>1 0 0</fdir1>
+  </gazebo>
+  <gazebo reference="left_rear_wheel">
+    <mu1>1000000000000000.0</mu1>
+    <mu2>1000000000000000.0</mu2>
+    <kp>1000000000000.0</kp>
+    <kd>10.0</kd>
+    <minDepth>0.001</minDepth>
+    <maxVel>0.1</maxVel>
+    <fdir1>1 0 0</fdir1>
+  </gazebo>
+  <gazebo reference="right_rear_wheel">
+    <mu1>1000000000000000.0</mu1>
+    <mu2>1000000000000000.0</mu2>
+    <kp>1000000000000.0</kp>
+    <kd>10.0</kd>
+    <minDepth>0.001</minDepth>
+    <maxVel>0.1</maxVel>
+    <fdir1>1 0 0</fdir1>
+  </gazebo>
+  <!-- ros2_control Gazebo plugins -->
   <gazebo>
-    <plugin name='diff_drive' filename='libgazebo_ros_diff_drive.so'>
-      <!-- Wheel Information -->
-      <left_joint>left_front_joint</left_joint>
-      <right_joint>right_front_joint</right_joint>
-      <wheel_separation>0.5715</wheel_separation>
-      <wheel_diameter>0.1524</wheel_diameter>
-      <!-- Limits -->
-      <max_wheel_torque>200</max_wheel_torque>
-      <max_wheel_acceleration>10.0</max_wheel_acceleration>
-      <!-- Odometry Output -->
-      <odometry_frame>odom</odometry_frame>
-      <robot_base_frame>base_link</robot_base_frame>
-      <publish_odom>true</publish_odom>
-      <publish_odom_tf>true</publish_odom_tf>
-      <publish_wheel_tf>true</publish_wheel_tf>
+    <plugin filename="gz_ros2_control-system" name="gz_ros2_control::GazeboSimROS2ControlPlugin">
+      <parameters>$(find robomagellan_controller)/config/robomagellan_controllers.yaml</parameters>
     </plugin>
   </gazebo>

File: ros2_ws/src/robomagellan_description/urdf/robomagellan.urdf.xacro (robot description, xacro)
@@ -4,7 +4,7 @@
   <xacro:arg name="is_sim" default="true"/>
   <!-- Include Gazebo parameters -->
- <!-- <xacro:include filename="$(find robomagellan_description)/urdf/gazebo.xacro"/> -->
-  <!-- Include ros2_contol plugins -->
- <!-- <xacro:include filename="$(find robomagellan_description)/urdf/ros2_control.xacro"/> -->
+  <xacro:include filename="$(find robomagellan_description)/urdf/gazebo.xacro"/>
+  <!-- Include ros2_contol plugins/interfaces -->
+  <xacro:include filename="$(find robomagellan_description)/urdf/ros2_control.xacro"/>
   <!-- Inertial Macros -->
   <xacro:macro name="inertial_box" params="mass x y z">

File: ros2_ws/src/robomagellan_description/urdf/ros2_control.xacro (robot description, xacro)
@@ -2,3 +2,34 @@
 <robot xmlns:xacro="http://www.ros.org/wiki/xacro" name="robot">
   <ros2_control name="RobotSystem" type="system">
+    <!-- ros2_control plugin for Gazebo -->
+    <xacro:if value="$(arg is_sim)">
+      <hardware>
+        <plugin>gz_ros2_control/GazeboSimSystem</plugin>
+      </hardware>
+    </xacro:if>
+    <!-- ros2_control plugin for the real robot -->
+    <xacro:unless value="$(arg is_sim)">
+      <hardware>
+        <plugin>robomagellan_firmware/RobomagellanInterface</plugin>
+        <param name="port">/dev/ttyUSB0</param>
+      </hardware>
+    </xacro:unless>
+    <!-- ros2_control common interfaces -->
+    <joint name="left_front_joint">
+      <command_interface name="velocity">
+        <param name="min">-1</param>
+        <param name="max">1</param>
+      </command_interface>
+      <state_interface name="position"/>
+      <state_interface name="velocity"/>
+    </joint>
+    <joint name="right_front_joint">
+      <command_interface name="velocity">
+        <param name="min">-1</param>
+        <param name="max">1</param>
+      </command_interface>
+      <state_interface name="position"/>
+      <state_interface name="velocity"/>
+    </joint>
+  </ros2_control>
 </robot>

Commit message: robomagellan_description - 0 Torsional Friction
Because we're using the Bullet Featherstone physics engine to support
mimic joints this commit sets the ground plane and robot wheels'
torsional friction coefficients to 0 so the robot can turn into place.

Signed-off-by: Bryant Pong <rcxking@gmail.com>

File: ros2_ws/src/robomagellan_description/urdf/gazebo.xacro (robot description, xacro)
@@ -1,41 +1,32 @@
 <?xml version="1.0"?>
 <robot name="robot" xmlns:xacro="http://www.ros.org/wiki/xacro">
-  <!-- Wheel links -->
-  <gazebo reference="left_front_wheel">
-    <mu1>1000000000000000.0</mu1>
-    <mu2>1000000000000000.0</mu2>
-    <kp>1000000000000.0</kp>
-    <kd>10.0</kd>
-    <minDepth>0.001</minDepth>
-    <maxVel>0.1</maxVel>
-    <fdir1>1 0 0</fdir1>
-  </gazebo>
-  <gazebo reference="right_front_wheel">
-    <mu1>1000000000000000.0</mu1>
-    <mu2>1000000000000000.0</mu2>
-    <kp>1000000000000.0</kp>
-    <kd>10.0</kd>
-    <minDepth>0.001</minDepth>
-    <maxVel>0.1</maxVel>
-    <fdir1>1 0 0</fdir1>
-  </gazebo>
-  <gazebo reference="left_rear_wheel">
-    <mu1>1000000000000000.0</mu1>
-    <mu2>1000000000000000.0</mu2>
-    <kp>1000000000000.0</kp>
-    <kd>10.0</kd>
-    <minDepth>0.001</minDepth>
-    <maxVel>0.1</maxVel>
-    <fdir1>1 0 0</fdir1>
-  </gazebo>
-  <gazebo reference="right_rear_wheel">
-    <mu1>1000000000000000.0</mu1>
-    <mu2>1000000000000000.0</mu2>
-    <kp>1000000000000.0</kp>
-    <kd>10.0</kd>
-    <minDepth>0.001</minDepth>
-    <maxVel>0.1</maxVel>
-    <fdir1>1 0 0</fdir1>
-  </gazebo>
+  <!-- Macro for setting Gazebo wheel parameters -->
+  <xacro:macro name="gazebo_wheel" params="prefix suffix">
+    <gazebo reference="${prefix}_${suffix}_wheel">
+      <mu1>1.0</mu1>
+      <mu2>0.0</mu2>
+      <kp>1000000000000.0</kp>
+      <kd>1.0</kd>
+      <minDepth>0.001</minDepth>
+      <maxVel>0.1</maxVel>
+      <fdir1>1 0 0</fdir1>
+      <!-- Bullet Featherstone engine: Need to set torsional friction to 0. -->
+      <!-- https://github.com/gazebosim/gz-physics/issues/697#issuecomment-2445495247 -->
+      <collision>
+        <surface>
+          <friction>
+            <torsional>
+              <coefficient>0.0</coefficient>
+            </torsional>
+          </friction>
+        </surface>
+      </collision>
+    </gazebo>
+  </xacro:macro>
+  <!-- Gazebo wheel parameters -->
+  <xacro:gazebo_wheel prefix="left" suffix="front"/>
+  <xacro:gazebo_wheel prefix="left" suffix="rear"/>
+  <xacro:gazebo_wheel prefix="right" suffix="front"/>
+  <xacro:gazebo_wheel prefix="right" suffix="rear"/>
   <!-- ros2_control Gazebo plugins -->
   <gazebo>

Commit message: IMU - Adding Simulated IMU
This commit adds a simulated IMU to the Gazebo robot model.  The IMU
data can be viewed by echoing the topic `/imu/out`.

Signed-off-by: Bryant Pong <rcxking@gmail.com>

File: ros2_ws/src/robomagellan_description/urdf/gazebo.xacro (robot description, xacro)
@@ -34,4 +34,58 @@
       <parameters>$(find robomagellan_controller)/config/robomagellan_controllers.yaml</parameters>
     </plugin>
+    <!-- Simulated IMU -->
+    <plugin filename="gz-sim-imu-system" name="gz::sim::systems::Imu">
+    </plugin>
+  </gazebo>
+  <!-- Simulated IMU parameters -->
+  <gazebo reference="imu_link">
+    <sensor name="imu" type="imu">
+      <always_on>true</always_on>
+      <update_rate>100</update_rate>
+      <gz_frame_id>imu_link</gz_frame_id>
+      <topic>imu</topic>
+      <imu>
+        <angular_velocity>
+          <x>
+            <noise type="gaussian">
+              <mean>0.0</mean>
+              <stddev>2e-4</stddev>
+            </noise>
+          </x>
+          <y>
+            <noise type="gaussian">
+              <mean>0.0</mean>
+              <stddev>2e-4</stddev>
+            </noise>
+          </y>
+          <z>
+            <noise type="gaussian">
+              <mean>0.0</mean>
+              <stddev>2e-4</stddev>
+            </noise>
+          </z>
+        </angular_velocity>
+        <linear_acceleration>
+          <x>
+            <noise type="gaussian">
+              <mean>0.0</mean>
+              <stddev>1.7e-2</stddev>
+            </noise>
+          </x>
+          <y>
+            <noise type="gaussian">
+              <mean>0.0</mean>
+              <stddev>1.7e-2</stddev>
+            </noise>
+          </y>
+          <z>
+            <noise type="gaussian">
+              <mean>0.0</mean>
+              <stddev>1.7e-2</stddev>
+            </noise>
+          </z>
+        </linear_acceleration>
+      </imu>
+    </sensor>
   </gazebo>
 </robot>

File: ros2_ws/src/robomagellan_description/urdf/robomagellan.urdf.xacro (robot description, xacro)
@@ -154,3 +154,32 @@
   <xacro:wheel prefix="right" suffix="front" reflectx="1" reflecty="-1" mimic_wheel="false"/>
   <xacro:wheel prefix="right" suffix="rear" reflectx="-1" reflecty="-1" mimic_wheel="true"/>
+  <!-- Simulated IMU (centered on robot's origin) -->
+  <link name="imu_link">
+    <inertial>
+      <origin xyz="0 0 0" rpy="0 0 0"/>
+      <mass value="0.0005"/>
+      <!-- TODO: Need dimensions of IMU -->
+      <inertia ixx="1.46176048428261E-08" ixy="1.40015117949421E-10" ixz="-1.9963387293740E-12" iyy="8.59662482954888E-09" iyz="7.52375112767959E-12" izz="2.30279421279312E-08" />
+    </inertial>
+    <visual>
+      <origin xyz="0 0 0" rpy="0 0 0"/>
+      <geometry>
+        <!-- TODO: Need dimensions of IMU -->
+        <box size="0.001 0.001 0.001"/>
+      </geometry>
+    </visual>
+    <collision>
+      <origin xyz="0 0 0" rpy="0 0 0"/>
+      <geometry>
+        <!-- TODO: Need dimensions of IMU -->
+        <box size="0.001 0.001 0.001"/>
+      </geometry>
+    </collision>
+  </link>
+  <joint name="imu_joint" type="fixed">
+    <origin xyz="0 0 0" rpy="0 0 0"/>
+    <parent link="base_link"/>
+    <child link="imu_link"/>
+    <axis xyz="0 0 0"/>
+  </joint>
 </robot>
